File: a8_garaj_extenter.kicad_pcb (KiCad board)
At the start: 2 copper layers, 85 x 45 mm, 48 parts, among them IC1 TCMT1100, IC10 TCMT1100, IC11 TCMT1100, IC12 TCMT1100, IC13 TCMT1100, IC14 TCMT1100, IC2 TCMT1100, IC3 TCMT1100, IC4 TCMT1100, IC5 TCMT1100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

Commit message: Update a8_garaj_extenter.kicad_pcb
Parts:
- added C1: C, Capacitor_SMD:C_1206_3216Metric_Pad1.33x1.80mm_HandSolder, F.Cu at (129.1, 103.2)
Connections:
- J1 pad 4: 3v3 -> unconnected-(J1-Pin_4-Pad4)
Routing:
- net SCL: track 0.00 -> 35.2 mm, vias 0 -> 1
- net SDA: track 2.83 -> 30.2 mm, vias 0 -> 1
- net 3v3: track 140.7 -> 148.1 mm
- net GNDREF: track 21.5 -> 22.5 mm, vias 16 -> 17
Other:
- outline, holes or cut-outs redrawn
- board text added: "12V"
- board text added: "GND"
- board text added: "NC"
- board text added: "SCL"
- board text added: "SDA"
